Commit message: fixed virtual joint bug

File: ynx_bringup/srdf/nex10/nex10.srdf_macro.xacro (robot description, xacro)
@@ -5,5 +5,5 @@
       <chain base_link="${tf_prefix}base_link" tip_link="${tf_prefix}tool0" />
     </group>
-    <virtual_joint name="virtual_joint" type="fixed" parent_frame="world" child_link="${tf_prefix}base_link"/>
+    <virtual_joint name="virtual_joint" type="fixed" parent_frame="world" child_link="${tf_prefix}mount_point"/>
     <group_state name="home" group="${tf_prefix}manipulator">
       <joint name="${tf_prefix}joint_1" value="0" />

File: ynx_description/urdf/nex10/nex10.urdf.xacro (robot description, xacro)
@@ -11,5 +11,4 @@
   <xacro:include filename="$(find ynx_description)/urdf/nex10/nex10.urdf_macro.xacro" />
   <xacro:include filename="$(find ynx_hardware_interface)/config/nex10/nex10.ros2_control_macro.xacro" />
-  <link name="world" />
   <xacro:nex10_urdf_macro tf_prefix="$(arg tf_prefix)"/>
   <xacro:nex10_ros2_control_macro tf_prefix="$(arg tf_prefix)" use_mock_hardware="$(arg use_mock_hardware)" ip="$(arg ip)" port="$(arg port)"/>

File: ynx_description/urdf/nex10/nex10.urdf_macro.xacro (robot description, xacro)
@@ -3,4 +3,5 @@
   <xacro:macro name="nex10_urdf_macro" params="tf_prefix">
     <!-- Links -->
+    <link name="${tf_prefix}mount_point"/>
     <link name="${tf_prefix}base_link"/>
     <link name="${tf_prefix}link_0">
@@ -140,5 +141,5 @@
     <joint name="${tf_prefix}base_joint" type="fixed">
       <origin xyz="0 0 0" rpy="0 0 0" />
-      <parent link="world" />
+      <parent link="${tf_prefix}mount_point" />
       <child link="${tf_prefix}base_link" />
     </joint>
